File: Breadboard Power Supply.kicad_pcb (KiCad board)
At the start: 2 copper layers, 28.7 x 52.3 mm, 19 parts, among them J1 Barrel_Jack_Switch, J2 Screw_Terminal_01x02, J3 Conn_01x03_Male, J4 Conn_01x02_Male, J5 Screw_Terminal_01x02, J6 Conn_01x02_Male, J7 Conn_01x03_Male, U1 LM317_TO-220, U2 LM7805_TO220

Commit message: Add files via upload
Parts:
- moved J4 45.8 mm to (120.9, 66.3)
- moved J6 45.8 mm to (120.9, 112.1)
Connections:
- J2 pad 2: /PWR_output -> /PWR_OUT_TOP
- J3 pad 2: /PWR_output -> /PWR_OUT_TOP
- J4 pad 2: /PWR_output -> /PWR_OUT_TOP
- J5 pad 2: /PWR_output -> /PWR_OUT_BOT
- J6 pad 2: /PWR_output -> /PWR_OUT_BOT
- J7 pad 2: /PWR_output -> /PWR_OUT_BOT
Routing:
- net /PWR_output: track 91.7 -> 0.00 mm
- net /PWR_OUT_BOT: track 0.00 -> 23.3 mm
- net /PWR_OUT_TOP: track 0.00 -> 21.5 mm
- net /5V: track 56.7 -> 62.2 mm
- net /3.3v: track 64.9 -> 69.0 mm, vias 1 -> 3
- net /PWR_input: track 17.9 -> 15.7 mm
- net Net-(D1-Pad2): track 9.84 -> 11.7 mm, vias 0 -> 1
- net Net-(R2-Pad1): track 24.9 -> 26.2 mm

Commit message: Contains  fix of the design bug
video course contains  fix of the design bug
Parts:
- R1: value 330 -> 560
- moved J6 0.05 mm to (120.9, 112.1)
Routing:
- net /5V: track 62.2 -> 56.7 mm
- net /3.3v: track 69.0 -> 64.9 mm, vias 3 -> 1
- net /PWR_input: track 15.7 -> 17.9 mm
- net Net-(D1-Pad2): track 11.7 -> 9.84 mm, vias 1 -> 0
- net Net-(R2-Pad1): track 26.2 -> 24.9 mm
