File: Breadboard Power Supply.kicad_sch (KiCad schematic)
At the start: 17 parts, among them J1 Barrel_Jack_Switch, J2 Screw_Terminal_01x02, J3 Conn_01x03_Male, J4 Conn_01x02_Male, J5 Screw_Terminal_01x02, J6 Conn_01x02_Male, J7 Conn_01x03_Male, U1 LM317_TO-220, U2 LM7805_TO220

Commit message: Add files via upload
Connections:
- net PWR_output renamed PWR_OUT_BOT
- net PWR_OUT_BOT: no longer J2.2 (Pin_2), J3.2 (Pin_2), J4.2 (Pin_2)
- new net PWR_OUT_TOP: J2.2 (Pin_2), J3.2 (Pin_2), J4.2 (Pin_2)
Changed lines of the file:
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@@
     (effects (font (size 1.27 1.27)) (justify left bottom))
   )
+  (label "PWR_OUT_BOT" (at 189.23 61.468 180)
+    (effects (font (size 1.27 1.27)) (justify right bottom))
+  )
   (label "5V" (at 195.834 52.324 180)
+    (effects (font (size 1.27 1.27)) (justify right bottom))
+  )
+  (label "PWR_OUT_TOP" (at 185.928 110.236 180)
     (effects (font (size 1.27 1.27)) (justify right bottom))
   )
@@
     (effects (font (size 1.27 1.27)) (justify left bottom))
   )
-  (label "PWR_output" (at 185.928 110.49 0)
-    (effects (font (size 1.27 1.27)) (justify left bottom))
-  )
   (label "3.3v" (at 121.666 101.346 0)
     (effects (font (size 1.27 1.27)) (justify left bottom))
@@
     (effects (font (size 1.27 1.27)) (justify left bottom))
   )
-  (label "PWR_output" (at 189.23 60.198 180)
-    (effects (font (size 1.27 1.27)) (justify right bottom))
-  )
   (label "5V" (at 141.986 46.736 0)

Commit message: Contains  fix of the design bug
video course contains  fix of the design bug
Parts:
- R1: value 330 -> 560
Changed lines of the file:
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@@
   (title_block
     (title "Learning KiCad with a simple project")
-    (date "2021-07-12")
-    (rev "1")
+    (date "2021-12-08")
+    (rev "2")
     (company "Tech Explorations")
   )
@@
     (effects (font (size 1.27 1.27)) (justify left bottom))
   )
-  (label "PWR_OUT_BOT" (at 189.23 61.468 180)
-    (effects (font (size 1.27 1.27)) (justify right bottom))
-  )
   (label "5V" (at 195.834 52.324 180)
     (effects (font (size 1.27 1.27)) (justify right bottom))
   )
-  (label "PWR_OUT_TOP" (at 185.928 110.236 180)
-    (effects (font (size 1.27 1.27)) (justify right bottom))
-  )
   (label "5V" (at 193.802 101.346 180)
     (effects (font (size 1.27 1.27)) (justify right bottom))
@@
     (effects (font (size 1.27 1.27)) (justify left bottom))
   )
+  (label "PWR_OUT_BOT" (at 189.23 60.452 180)
+    (effects (font (size 1.27 1.27)) (justify right bottom))
+  )
   (label "12V" (at 88.9 46.736 0)
     (effects (font (size 1.27 1.27)) (justify left bottom))
@@
   )
   (label "3.3v" (at 195.834 57.404 180)
+    (effects (font (size 1.27 1.27)) (justify right bottom))
+  )
+  (label "PWR_OUT_TOP" (at 185.928 112.014 180)
     (effects (font (size 1.27 1.27)) (justify right bottom))
   )
@@
       (effects (font (size 1.27 1.27)) (justify right))
     )
-    (property "Value" "330" (id 1) (at 55.88 111.5059 0)
+    (property "Value" "560" (id 1) (at 55.88 111.5059 0)
       (effects (font (size 1.27 1.27)) (justify right))
     )
@@
     )
     (path "/444835ed-df3b-4c9b-8dd4-e0c752098dee"
-      (reference "R1") (unit 1) (value "330") (footprint "Resistor_THT:R_Axial_DIN0204_L3.6mm_D1.6mm_P7.62mm_Horizontal")
+      (reference "R1") (unit 1) (value "560") (footprint "Resistor_THT:R_Axial_DIN0204_L3.6mm_D1.6mm_P7.62mm_Horizontal")
     )
     (path "/6244ec7e-f6fa-4582-8639-1449847d9d8f"
